Commit message: Update .gitignore and refactor hermes_sim SDF model for improved simulation compatibility

File: urdf/hermes_sim.sdf.xacro (robot description, xacro)
@@ -1,237 +1,312 @@
-<?xml version="1.0"?>
-<!--
-  hermes_sim.sdf.xacro
-  ====================
-  Simulation SDF model for the HERMES differential-drive robot.
-  Designed for Gazebo Harmonic (gz-sim) with ROS 2 Jazzy.
-  All primary dimensions are declared as <xacro:property> at the top of
-  the file.  Derived values (half-lengths, offsets, inertias) are computed
-  from those primaries so that a single edit propagates everywhere.
-  TF tree produced at runtime
-  ===========================
-    odom  <- (DiffDrive plugin via /tf bridge)
-      base_footprint   (virtual, at ground level)
-        base_link      (cube body centre, body_z m AGL)
-          wheel_left_link
-          wheel_right_link
-          caster_link      (front caster)
-          laser_frame      (LiDAR on top of body)
-          camera_frame     (camera at front-top of body)
-  Topics
-  ======
-    /cmd_vel       geometry_msgs/Twist    => drive command  (ROS => gz)
-    /odom          nav_msgs/Odometry      <= wheel odometry (gz => ROS)
-    /scan          sensor_msgs/LaserScan  <= 360 deg LiDAR  (gz => ROS)
-    /tf            tf2_msgs/TFMessage     <= odom->base_footprint (gz => ROS)
-    /joint_states  sensor_msgs/JointState <= wheel joints   (gz => ROS)
--->
-<sdf version="1.9" xmlns:xacro="http://www.ros.org/wiki/xacro">
-  <!-- ════════════════════════════════════════════════════════════════════════
-       Primary dimensions  (edit here; everything else is derived)
-       ════════════════════════════════════════════════════════════════════════ -->
-  <!-- Body: cube 5.5 in per side -->
-  <xacro:property name="body_size" value="0.1397"/>   <!-- m  (5.5 in) -->
-  <xacro:property name="body_mass" value="5.0"/>       <!-- kg -->
-  <!-- Drive wheels: 2.6 in diameter, 0.7 in wide -->
-  <xacro:property name="wheel_radius" value="0.0330"/> <!-- m  (1.3 in) -->
-  <xacro:property name="wheel_width"  value="0.0178"/> <!-- m  (0.7 in) -->
-  <xacro:property name="wheel_mass"   value="0.5"/>    <!-- kg -->
-  <!-- Caster: passive front sphere -->
-  <xacro:property name="caster_mass"  value="0.1"/>    <!-- kg -->
-  <!-- ── Derived geometry ──────────────────────────────────────────────────── -->
-  <xacro:property name="body_half"     value="${body_size   / 2}"/>
-  <xacro:property name="caster_radius" value="${wheel_radius / 2}"/>
-  <!-- wheel_y : lateral distance from base_link centre to wheel centre -->
-  <xacro:property name="wheel_y"   value="${body_half + wheel_width / 2}"/>
-  <!-- wheel_sep : centre-to-centre track width (used by DiffDrive plugin) -->
-  <xacro:property name="wheel_sep" value="${2 * wheel_y}"/>
-  <!-- body_z : height of base_link centre above ground when spawned -->
-  <!--          = wheel_radius + body_half                           -->
-  <xacro:property name="body_z"    value="${wheel_radius + body_half}"/>
-  <!-- wheel_z : z of wheel axle relative to base_link (= -body_half) -->
-  <xacro:property name="wheel_z"   value="${-body_half}"/>
-  <!-- caster_x : forward offset of caster centre from base_link -->
-  <xacro:property name="caster_x"  value="${body_half - caster_radius}"/>
-  <!-- caster_z : z of caster centre relative to base_link        -->
-  <xacro:property name="caster_z"  value="${caster_radius - body_z}"/>
-  <!-- ── Derived inertias ──────────────────────────────────────────────────── -->
-  <!-- Solid cube:     I = m * s² / 6                                          -->
-  <xacro:property name="body_ixx"
-      value="${body_mass * body_size**2 / 6}"/>
-  <!-- Solid cylinder: Ixx = Iyy = m*(3r²+h²)/12,  Izz = m*r²/2              -->
-  <xacro:property name="wheel_ixx"
-      value="${wheel_mass * (3 * wheel_radius**2 + wheel_width**2) / 12}"/>
-  <xacro:property name="wheel_izz"
-      value="${wheel_mass * wheel_radius**2 / 2}"/>
-  <!-- Solid sphere:   I = 2*m*r² / 5                                          -->
-  <xacro:property name="caster_ixx"
-      value="${2 * caster_mass * caster_radius**2 / 5}"/>
-  <!-- ════════════════════════════════════════════════════════════════════════
-       Wheel macro  —  one link + one revolute joint
-         prefix : "left" or "right"
-         y_pos  : signed lateral offset from base_link centre (m)
-                  pass ${wheel_y} for left, ${-wheel_y} for right
-       ════════════════════════════════════════════════════════════════════════ -->
-  <xacro:macro name="wheel" params="prefix y_pos">
-    <link name="wheel_${prefix}_link">
-      <pose relative_to="base_link">0 ${y_pos} ${wheel_z} 1.5708 0 0</pose>
+<?xml version="1.0" ?>
+<sdf version="1.8" xmlns:xacro="http://ros.org/wiki/xacro">
+  <model name='hermes_robot' canonical_link='base_link'>
+    <!-- Define robot constants -->
+    <xacro:property name="base_width" value="0.31"/>
+    <xacro:property name="base_length" value="0.42"/>
+    <xacro:property name="base_height" value="0.18"/>
+    <xacro:property name="wheel_radius" value="0.10"/>
+    <xacro:property name="wheel_width" value="0.04"/>
+    <xacro:property name="wheel_ygap" value="0.025"/>
+    <xacro:property name="wheel_zoff" value="0.05"/>
+    <xacro:property name="wheel_xoff" value="0.12"/>
+    <xacro:property name="caster_xoff" value="0.14"/>
+    <!-- Define some commonly used intertial properties  -->
+    <xacro:macro name="box_inertia" params="m w h d">
       <inertial>
-        <mass>${wheel_mass}</mass>
+        <pose>0 0 0 ${pi/2} 0 ${pi/2}</pose>
+        <mass>${m}</mass>
         <inertia>
-          <ixx>${wheel_ixx}</ixx><ixy>0</ixy><ixz>0</ixz>
-          <iyy>${wheel_ixx}</iyy><iyz>0</iyz>
-          <izz>${wheel_izz}</izz>
+          <ixx>${(m/12) * (h*h + d*d)}</ixx>
+          <ixy>0.0</ixy>
+          <ixz>0.0</ixz>
+          <iyy>${(m/12) * (w*w + d*d)}</iyy>
+          <iyz>0.0</iyz>
+          <izz>${(m/12) * (w*w + h*h)}</izz>
         </inertia>
       </inertial>
-      <visual name="visual">
-        <geometry>
-          <cylinder>
-            <radius>${wheel_radius}</radius>
-            <length>${wheel_width}</length>
-          </cylinder>
-        </geometry>
-        <material>
-          <ambient>0.1 0.1 0.1 1</ambient>
-          <diffuse>0.1 0.1 0.1 1</diffuse>
-        </material>
-      </visual>
-      <collision name="collision">
-        <geometry>
-          <cylinder>
-            <radius>${wheel_radius}</radius>
-            <length>${wheel_width}</length>
-          </cylinder>
-        </geometry>
-        <surface>
-          <friction><ode><mu>1.0</mu><mu2>1.0</mu2></ode></friction>
-        </surface>
-      </collision>
-    </link>
-    <joint name="wheel_${prefix}_joint" type="revolute">
-      <parent>base_link</parent>
-      <child>wheel_${prefix}_link</child>
-      <axis>
-        <xyz expressed_in="__model__">0 1 0</xyz>
-        <limit><lower>-1e+16</lower><upper>1e+16</upper></limit>
-      </axis>
-    </joint>
-  </xacro:macro>
-  <!-- ════════════════════════════════════════════════════════════════════════
-       Model
-       ════════════════════════════════════════════════════════════════════════ -->
-  <model name="hermes">
-    <!-- ── base_link (cube body) ─────────────────────────────────────────── -->
-    <link name="base_link">
+    </xacro:macro>
+    <xacro:macro name="cylinder_inertia" params="m r h">
       <inertial>
-        <mass>${body_mass}</mass>
+        <pose>0 0 0 ${pi/2} 0 0</pose>
+        <mass>${m}</mass>
         <inertia>
-          <ixx>${body_ixx}</ixx><ixy>0</ixy><ixz>0</ixz>
-          <iyy>${body_ixx}</iyy><iyz>0</iyz>
-          <izz>${body_ixx}</izz>
+          <ixx>${(m/12) * (3*r*r + h*h)}</ixx>
+          <ixy>0.0</ixy>
+          <ixz>0.0</ixz>
+          <iyy>${(m/12) * (3*r*r + h*h)}</iyy>
+          <iyz>0.0</iyz>
+          <izz>${(m/2) * (r*r)}</izz>
         </inertia>
       </inertial>
-      <visual name="visual">
-        <geometry>
-          <box><size>${body_size} ${body_size} ${body_size}</size></box>
-        </geometry>
-        <material>
-          <ambient>0.3 0.3 0.3 1</ambient>
-          <diffuse>0.3 0.3 0.3 1</diffuse>
-        </material>
-      </visual>
-      <collision name="collision">
-        <geometry>
-          <box><size>${body_size} ${body_size} ${body_size}</size></box>
-        </geometry>
-      </collision>
-    </link>
-    <!-- ── base_footprint (virtual, at ground level) ─────────────────────── -->
-    <link name="base_footprint">
-      <pose relative_to="base_link">0 0 ${-body_z} 0 0 0</pose>
-    </link>
-    <joint name="base_footprint_joint" type="fixed">
-      <parent>base_link</parent>
-      <child>base_footprint</child>
-    </joint>
-    <!-- ── Drive wheels ──────────────────────────────────────────────────── -->
-    <xacro:wheel prefix="left"  y_pos="${wheel_y}"/>
-    <xacro:wheel prefix="right" y_pos="${-wheel_y}"/>
-    <!-- ── Caster wheel (front, passive, zero friction) ──────────────────── -->
-    <link name="caster_link">
-      <pose relative_to="base_link">${caster_x} 0 ${caster_z} 0 0 0</pose>
+    </xacro:macro>
+    <xacro:macro name="sphere_inertia" params="m r">
       <inertial>
-        <mass>${caster_mass}</mass>
+        <mass>${m}</mass>
         <inertia>
-          <ixx>${caster_ixx}</ixx><ixy>0</ixy><ixz>0</ixz>
-          <iyy>${caster_ixx}</iyy><iyz>0</iyz>
-          <izz>${caster_ixx}</izz>
+          <ixx>${(2/5) * m * (r*r)}</ixx>
+          <ixy>0.0</ixy>
+          <ixz>0.0</ixz>
+          <iyy>${(2/5) * m * (r*r)}</iyy>
+          <iyz>0.0</iyz>
+          <izz>${(2/5) * m * (r*r)}</izz>
         </inertia>
       </inertial>
-      <visual name="visual">
-        <geometry>
-          <sphere><radius>${caster_radius}</radius></sphere>
+    </xacro:macro>
+    <!-- Robot Base -->
+    <link name='base_link'>
+      <must_be_base_link>true</must_be_base_link>
+      <visual name="base_link_visual">
+        <geometry>
+          <box><size>
+            ${base_length} ${base_width} ${base_height}
+          </size></box>
         </geometry>
         <material>
-          <ambient>0.6 0.6 0.6 1</ambient>
-          <diffuse>0.6 0.6 0.6 1</diffuse>
+          <ambient>0 1 1 1</ambient>
+          <diffuse>0 1 1 1</diffuse>
         </material>
       </visual>
-      <collision name="collision">
-        <geometry>
-          <sphere><radius>${caster_radius}</radius></sphere>
-        </geometry>
-        <surface>
-          <friction><ode><mu>0.0</mu><mu2>0.0</mu2></ode></friction>
-        </surface>
-      </collision>
+      <collision name="base_link_collision">
+        <geometry>
+          <box><size>
+            ${base_length} ${base_width} ${base_height}
+          </size></box>
+        </geometry>
+      </collision>
+    </link>
+    <!-- Robot Footprint -->
+    <link name='base_footprint'>
+      <pose relative_to="base_joint"/>
+      <xacro:box_inertia m="15" w="${base_width}" d="${base_length}" h="${base_height}"/>
+    </link>
+    <joint name='base_joint' type='fixed'>
+      <parent>base_link</parent>
+      <child>base_footprint</child>
+      <pose relative_to="base_link">0.0 0.0 ${-(wheel_radius+wheel_zoff)} 0 0 0</pose>
+    </joint>
+    <!-- Wheels -->
+    <xacro:macro name="wheel" params="prefix x_reflect y_reflect">
+      <link name="${prefix}_link">
+        <pose relative_to="${prefix}_joint"/>
+        <visual name="${prefix}_link_visual">
+          <pose relative_to="${prefix}_link">0 0 0 ${pi/2} 0 0</pose>
+          <geometry>
+            <cylinder>
+              <radius>${wheel_radius}</radius>
+              <length>${wheel_width}</length>
+            </cylinder>
+          </geometry>
+          <material>
+            <ambient>0.3 0.3 0.3 1.0</ambient>
+            <diffuse>0.7 0.7 0.7 1.0</diffuse>
+          </material>
+        </visual>
+        <collision name="${prefix}_link_collision">
+          <pose relative_to="${prefix}_link">0 0 0 ${pi/2} 0 0</pose>
+          <geometry>
+            <cylinder>
+              <radius>${wheel_radius}</radius>
+              <length>${wheel_width}</length>
+            </cylinder>
+          </geometry>
+        </collision>
+        <xacro:cylinder_inertia m="0.5" r="${wheel_radius}" h="${wheel_width}"/>
+      </link>
+      <joint name="${prefix}_joint" type="revolute">
+        <parent>base_link</parent>
+        <child>${prefix}_link</child>
+        <pose relative_to="base_link">${x_reflect*wheel_xoff} ${y_reflect*(base_width/2+wheel_ygap)} ${-wheel_zoff} 0 0 0</pose>
+        <axis>
+          <xyz>0 1 0</xyz>
+          <limit>
+            <lower>-inf</lower>
+            <upper>inf</upper>
+          </limit>
+        </axis>
+      </joint>
+    </xacro:macro>
+    <xacro:wheel prefix="drivewhl_l" x_reflect="-1" y_reflect="1" />
+    <xacro:wheel prefix="drivewhl_r" x_reflect="-1" y_reflect="-1" />
+    <link name="front_caster">
+      <pose relative_to="caster_joint"/>
+      <visual name="front_caster_visual">
+        <geometry>
+          <sphere>
+            <radius>${(wheel_radius+wheel_zoff-(base_height/2))}</radius>
+          </sphere>
+        </geometry>
+        <material>
+          <ambient>0 1 1 1</ambient>
+          <diffuse>0 1 1 1</diffuse>
+        </material>
+      </visual>
+      <collision name="front_caster_collision">
+        <geometry>
+          <sphere>
+            <radius>${(wheel_radius+wheel_zoff-(base_height/2))}</radius>
+          </sphere>
+        </geometry>
+        <surface><friction><ode>
+          <mu>0.001</mu>
+          <mu2>0.001</mu2>
+        </ode></friction></surface>
+      </collision>
+      <xacro:sphere_inertia m="0.5" r="${(wheel_radius+wheel_zoff-(base_height/2))}"/>
     </link>
     <joint name="caster_joint" type="fixed">
       <parent>base_link</parent>
-      <child>caster_link</child>
-    </joint>
-    <!-- ── laser_frame (2-D LiDAR, top of body) ─────────────────────────── -->
-    <link name="laser_frame">
-      <pose relative_to="base_link">0 0 ${body_half} 0 0 0</pose>
-      <inertial>
-        <mass>0.1</mass>
-        <inertia>
-          <ixx>0.00001</ixx><ixy>0</ixy><ixz>0</ixz>
-          <iyy>0.00001</iyy><iyz>0</iyz>
-          <izz>0.00001</izz>
-        </inertia>
-      </inertial>
-      <visual name="visual">
-        <geometry>
-          <cylinder><radius>0.04</radius><length>0.04</length></cylinder>
-        </geometry>
-        <material>
-          <ambient>0.0 0.4 0.8 1</ambient>
-          <diffuse>0.0 0.4 0.8 1</diffuse>
-        </material>
-      </visual>
-      <collision name="collision">
-        <geometry>
-          <cylinder><radius>0.04</radius><length>0.04</length></cylinder>
-        </geometry>
-      </collision>
-      <!-- 2-D LiDAR (360 deg, 10 Hz, 12 m range) -->
+      <child>front_caster</child>
+      <pose relative_to="base_link">${caster_xoff} 0.0 ${-(base_height/2)} 0 0 0</pose>
+    </joint>
+    <joint name='imu_joint' type='fixed'>
+      <parent>base_link</parent>
+      <child>imu_link</child>
+      <pose relative_to="base_link">0.0 0.0 0.01 0 0 0</pose>
+    </joint>
+    <link name='imu_link'>
+      <pose relative_to="imu_joint"/>
+      <visual name="imu_link_visual">
+        <geometry>
+          <box><size>
+            0.1 0.1 0.1
+          </size></box>
+        </geometry>
+      </visual>
+      <collision name="imu_link_collision">
+        <geometry>
+          <box><size>
+            0.1 0.1 0.1
+          </size></box>
+        </geometry>
+      </collision>
+      <xacro:box_inertia m="0.1" w="0.1" d="0.1" h="0.1"/>
+      <sensor name="imu_sensor" type="imu">
+        <always_on>true</always_on>
+        <update_rate>100</update_rate>
+        <visualize>true</visualize>
+        <topic>demo/imu</topic>
+        <gz_frame_id>imu_link</gz_frame_id>
+        <imu>
+          <angular_velocity>
+            <x>
+              <noise type="gaussian">
+                <mean>0.0</mean>
+                <stddev>2e-4</stddev>
+                <bias_mean>0.0000075</bias_mean>
+                <bias_stddev>0.0000008</bias_stddev>
+              </noise>
+            </x>
+            <y>
+              <noise type="gaussian">
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