Commit message: Update robot body, wheels, sensors per spec: 4.5x4.5x3in body, 1.3in wheel radius, 0.5in caster, lidar on top, remove IMU
Co-authored-by: numbersletter <41592985+numbersletter@users.noreply.github.com>

File: urdf/hermes_sim.sdf.xacro (robot description, xacro)
@@ -3,13 +3,22 @@
   <model name='hermes_robot' canonical_link='base_link'>
     <!-- Define robot constants -->
-    <xacro:property name="base_width" value="0.31"/>
-    <xacro:property name="base_length" value="0.42"/>
-    <xacro:property name="base_height" value="0.18"/>
-    <xacro:property name="wheel_radius" value="0.10"/>
-    <xacro:property name="wheel_width" value="0.04"/>
+    <!-- Body: 4.5x4.5 in x 3 in (converted to meters) -->
+    <xacro:property name="base_width" value="0.1143"/>
+    <xacro:property name="base_length" value="0.1143"/>
+    <xacro:property name="base_height" value="0.0762"/>
+    <!-- Wheels: radius 1.3 in, width 0.7 in (converted to meters) -->
+    <xacro:property name="wheel_radius" value="0.03302"/>
+    <xacro:property name="wheel_width" value="0.01778"/>
     <xacro:property name="wheel_ygap" value="0.025"/>
-    <xacro:property name="wheel_zoff" value="0.05"/>
-    <xacro:property name="wheel_xoff" value="0.12"/>
-    <xacro:property name="caster_xoff" value="0.14"/>
+    <xacro:property name="wheel_xoff" value="0.04"/>
+    <!-- Caster: radius 0.5 in (converted to meters) -->
+    <xacro:property name="caster_radius" value="0.0127"/>
+    <xacro:property name="caster_xoff" value="0.04"/>
+    <!-- wheel_zoff keeps drive wheels and caster both touching the ground -->
+    <!-- wheel_zoff = base_height/2 + caster_radius - wheel_radius -->
+    <xacro:property name="wheel_zoff" value="${base_height/2 + caster_radius - wheel_radius}"/>
+    <!-- Lidar: radius 1.5 in, length 0.8 in (converted to meters) -->
+    <xacro:property name="lidar_radius" value="0.0381"/>
+    <xacro:property name="lidar_length" value="0.02032"/>
     <!-- Define some commonly used intertial properties  -->
     <xacro:macro name="box_inertia" params="m w h d">
@@ -79,5 +88,5 @@
     <link name='base_footprint'>
       <pose relative_to="base_joint"/>
-      <xacro:box_inertia m="15" w="${base_width}" d="${base_length}" h="${base_height}"/>
+      <xacro:box_inertia m="2" w="${base_width}" d="${base_length}" h="${base_height}"/>
     </link>
     <joint name='base_joint' type='fixed'>
@@ -134,5 +143,5 @@
         <geometry>
           <sphere>
-            <radius>${(wheel_radius+wheel_zoff-(base_height/2))}</radius>
+            <radius>${caster_radius}</radius>
           </sphere>
         </geometry>
@@ -145,5 +154,5 @@
         <geometry>
           <sphere>
-            <radius>${(wheel_radius+wheel_zoff-(base_height/2))}</radius>
+            <radius>${caster_radius}</radius>
           </sphere>
         </geometry>
@@ -153,5 +162,5 @@
         </ode></friction></surface>
       </collision>
-      <xacro:sphere_inertia m="0.5" r="${(wheel_radius+wheel_zoff-(base_height/2))}"/>
+      <xacro:sphere_inertia m="0.5" r="${caster_radius}"/>
     </link>
     <joint name="caster_joint" type="fixed">
@@ -160,88 +169,4 @@
       <pose relative_to="base_link">${caster_xoff} 0.0 ${-(base_height/2)} 0 0 0</pose>
     </joint>
-    <joint name='imu_joint' type='fixed'>
-      <parent>base_link</parent>
-      <child>imu_link</child>
-      <pose relative_to="base_link">0.0 0.0 0.01 0 0 0</pose>
-    </joint>
-    <link name='imu_link'>
-      <pose relative_to="imu_joint"/>
-      <visual name="imu_link_visual">
-        <geometry>
-          <box><size>
-            0.1 0.1 0.1
-          </size></box>
-        </geometry>
-      </visual>
-      <collision name="imu_link_collision">
-        <geometry>
-          <box><size>
-            0.1 0.1 0.1
-          </size></box>
-        </geometry>
-      </collision>
-      <xacro:box_inertia m="0.1" w="0.1" d="0.1" h="0.1"/>
-      <sensor name="imu_sensor" type="imu">
-        <always_on>true</always_on>
-        <update_rate>100</update_rate>
-        <visualize>true</visualize>
-        <topic>demo/imu</topic>
-        <gz_frame_id>imu_link</gz_frame_id>
-        <imu>
-          <angular_velocity>
-            <x>
-              <noise type="gaussian">
-                <mean>0.0</mean>
-                <stddev>2e-4</stddev>
-                <bias_mean>0.0000075</bias_mean>
-                <bias_stddev>0.0000008</bias_stddev>
-              </noise>
-            </x>
-            <y>
-              <noise type="gaussian">
-                <mean>0.0</mean>
-                <stddev>2e-4</stddev>
-                <bias_mean>0.0000075</bias_mean>
-                <bias_stddev>0.0000008</bias_stddev>
-              </noise>
-            </y>
-            <z>
-              <noise type="gaussian">
-                <mean>0.0</mean>
-                <stddev>2e-4</stddev>
-                <bias_mean>0.0000075</bias_mean>
-                <bias_stddev>0.0000008</bias_stddev>
-              </noise>
-            </z>
-          </angular_velocity>
-          <linear_acceleration>
-            <x>
-              <noise type="gaussian">
-                <mean>0.0</mean>
-                <stddev>1.7e-2</stddev>
-                <bias_mean>0.1</bias_mean>
-                <bias_stddev>0.001</bias_stddev>
-              </noise>
-            </x>
-            <y>
-              <noise type="gaussian">
-                <mean>0.0</mean>
-                <stddev>1.7e-2</stddev>
-                <bias_mean>0.1</bias_mean>
-                <bias_stddev>0.001</bias_stddev>
-              </noise>
-            </y>
-            <z>
-              <noise type="gaussian">
-                <mean>0.0</mean>
-                <stddev>1.7e-2</stddev>
-                <bias_mean>0.1</bias_mean>
-                <bias_stddev>0.001</bias_stddev>
-              </noise>
-            </z>
-          </linear_acceleration>
-        </imu>
-      </sensor>
-    </link>
     <plugin filename="gz-sim-diff-drive-system" name="gz::sim::systems::DiffDrive">
       <!-- wheels -->
@@ -249,5 +174,5 @@
       <right_joint>drivewhl_r_joint</right_joint>
       <!-- kinematics -->
-      <wheel_separation>0.4</wheel_separation>
+      <wheel_separation>${base_width + 2*wheel_ygap}</wheel_separation>
       <wheel_radius>${wheel_radius}</wheel_radius>
       <!-- limits -->
@@ -269,5 +194,6 @@
       <parent>base_link</parent>
       <child>lidar_link</child>
-      <pose relative_to="base_link">0.0 0.0 0.12 0 0 0</pose>
+      <!-- Lidar sits right on top of the body: body_top + lidar_half_length -->
+      <pose relative_to="base_link">0.0 0.0 ${base_height/2 + lidar_length/2} 0 0 0</pose>
     </joint>
     <link name='lidar_link'>
@@ -276,6 +202,6 @@
         <geometry>
           <cylinder>
-            <radius>0.0508</radius>
-            <length>0.055</length>
+            <radius>${lidar_radius}</radius>
+            <length>${lidar_length}</length>
           </cylinder>
         </geometry>
@@ -284,10 +210,10 @@
         <geometry>
           <cylinder>
-            <radius>0.0508</radius>
-            <length>0.055</length>
+            <radius>${lidar_radius}</radius>
+            <length>${lidar_length}</length>
           </cylinder>
         </geometry>
       </collision>
-      <xacro:cylinder_inertia m="0.125" r="0.0508" h="0.055"/>
+      <xacro:cylinder_inertia m="0.125" r="${lidar_radius}" h="${lidar_length}"/>
       <sensor name="lidar" type="gpu_lidar">
         <always_on>true</always_on>
@@ -321,5 +247,5 @@
       <parent>base_link</parent>
       <child>camera_link</child>
-      <pose relative_to="base_link">0.215 0 0.05 0 0 0</pose>
+      <pose relative_to="base_link">${base_length/2} 0 0 0 0 0</pose>
     </joint>
     <link name='camera_link'>

Commit message: Add a launch to display robot, changed simulated robot parameters. Changed the bridge config so only necessary topics to closesly mimic real setup are shown (just clock, cmd_vel, scan), which means the diff_drive plugin (or the real controller) does not output odometry. All odometry from rf2o (lidar) which publishes tf odom->base_link and odometry over /odom_rf2o (configurable). When we do the full simulation, we may need to reconfigure rf2o so the odometry messages are passed in /odom.

File: urdf/hermes_sim.sdf.xacro (robot description, xacro)
@@ -3,13 +3,13 @@
   <model name='hermes_robot' canonical_link='base_link'>
     <!-- Define robot constants -->
-    <xacro:property name="base_width" value="0.31"/>
-    <xacro:property name="base_length" value="0.42"/>
-    <xacro:property name="base_height" value="0.18"/>
-    <xacro:property name="wheel_radius" value="0.10"/>
-    <xacro:property name="wheel_width" value="0.04"/>
-    <xacro:property name="wheel_ygap" value="0.025"/>
-    <xacro:property name="wheel_zoff" value="0.05"/>
-    <xacro:property name="wheel_xoff" value="0.12"/>
-    <xacro:property name="caster_xoff" value="0.14"/>
+    <xacro:property name="base_width" value="0.1143"/>
+    <xacro:property name="base_length" value="0.1143"/>
+    <xacro:property name="base_height" value="0.0762"/>
+    <xacro:property name="wheel_radius" value="0.03302"/>
+    <xacro:property name="wheel_width" value="0.01778"/>
+    <xacro:property name="wheel_ygap" value="0.01"/>
+    <xacro:property name="wheel_zoff" value="0.01778"/>
+    <xacro:property name="wheel_xoff" value="0.03"/>
+    <xacro:property name="caster_xoff" value="0.04"/>
     <!-- Define some commonly used intertial properties  -->
     <xacro:macro name="box_inertia" params="m w h d">
@@ -79,5 +79,5 @@
     <link name='base_footprint'>
       <pose relative_to="base_joint"/>
-      <xacro:box_inertia m="15" w="${base_width}" d="${base_length}" h="${base_height}"/>
+      <xacro:box_inertia m="2.0" w="${base_width}" d="${base_length}" h="${base_height}"/>
     </link>
     <joint name='base_joint' type='fixed'>
@@ -160,88 +160,4 @@
       <pose relative_to="base_link">${caster_xoff} 0.0 ${-(base_height/2)} 0 0 0</pose>
     </joint>
-    <joint name='imu_joint' type='fixed'>
-      <parent>base_link</parent>
-      <child>imu_link</child>
-      <pose relative_to="base_link">0.0 0.0 0.01 0 0 0</pose>
-    </joint>
-    <link name='imu_link'>
-      <pose relative_to="imu_joint"/>
-      <visual name="imu_link_visual">
-        <geometry>
-          <box><size>
-            0.1 0.1 0.1
-          </size></box>
-        </geometry>
-      </visual>
-      <collision name="imu_link_collision">
-        <geometry>
-          <box><size>
-            0.1 0.1 0.1
-          </size></box>
-        </geometry>
-      </collision>
-      <xacro:box_inertia m="0.1" w="0.1" d="0.1" h="0.1"/>
-      <sensor name="imu_sensor" type="imu">
-        <always_on>true</always_on>
-        <update_rate>100</update_rate>
-        <visualize>true</visualize>
-        <topic>demo/imu</topic>
-        <gz_frame_id>imu_link</gz_frame_id>
-        <imu>
-          <angular_velocity>
-            <x>
-              <noise type="gaussian">
-                <mean>0.0</mean>
-                <stddev>2e-4</stddev>
-                <bias_mean>0.0000075</bias_mean>
-                <bias_stddev>0.0000008</bias_stddev>
-              </noise>
-            </x>
-            <y>
-              <noise type="gaussian">
-                <mean>0.0</mean>
-                <stddev>2e-4</stddev>
-                <bias_mean>0.0000075</bias_mean>
-                <bias_stddev>0.0000008</bias_stddev>
-              </noise>
-            </y>
-            <z>
-              <noise type="gaussian">
-                <mean>0.0</mean>
-                <stddev>2e-4</stddev>
-                <bias_mean>0.0000075</bias_mean>
-                <bias_stddev>0.0000008</bias_stddev>
-              </noise>
-            </z>
-          </angular_velocity>
-          <linear_acceleration>
-            <x>
-              <noise type="gaussian">
-                <mean>0.0</mean>
-                <stddev>1.7e-2</stddev>
-                <bias_mean>0.1</bias_mean>
-                <bias_stddev>0.001</bias_stddev>
-              </noise>
-            </x>
-            <y>
-              <noise type="gaussian">
-                <mean>0.0</mean>
-                <stddev>1.7e-2</stddev>
-                <bias_mean>0.1</bias_mean>
-                <bias_stddev>0.001</bias_stddev>
-              </noise>
-            </y>
-            <z>
-              <noise type="gaussian">
-                <mean>0.0</mean>
-                <stddev>1.7e-2</stddev>
-                <bias_mean>0.1</bias_mean>
-                <bias_stddev>0.001</bias_stddev>
-              </noise>
-            </z>
-          </linear_acceleration>
-        </imu>
-      </sensor>
-    </link>
     <plugin filename="gz-sim-diff-drive-system" name="gz::sim::systems::DiffDrive">
       <!-- wheels -->
@@ -249,5 +165,5 @@
       <right_joint>drivewhl_r_joint</right_joint>
       <!-- kinematics -->
-      <wheel_separation>0.4</wheel_separation>
+      <wheel_separation>0.1343</wheel_separation>
       <wheel_radius>${wheel_radius}</wheel_radius>
       <!-- limits -->
@@ -255,9 +171,4 @@
       <!-- input -->
       <topic>/demo/cmd_vel</topic>
-      <!-- output -->
-      <odom_topic>/demo/odom</odom_topic>
-      <tf_topic>/tf</tf_topic>
-      <frame_id>odom</frame_id>
-      <child_frame_id>base_link</child_frame_id>
     </plugin>
     <plugin
@@ -269,5 +180,5 @@
       <parent>base_link</parent>
       <child>lidar_link</child>
-      <pose relative_to="base_link">0.0 0.0 0.12 0 0 0</pose>
+      <pose relative_to="base_link">0.0 0.0 0.04826 0 0 0</pose>
     </joint>
     <link name='lidar_link'>
@@ -276,6 +187,6 @@
         <geometry>
           <cylinder>
-            <radius>0.0508</radius>
-            <length>0.055</length>
+            <radius>0.021</radius>
+            <length>0.02032</length>
           </cylinder>
         </geometry>
@@ -284,10 +195,10 @@
         <geometry>
           <cylinder>
-            <radius>0.0508</radius>
-            <length>0.055</length>
+            <radius>0.021</radius>
+            <length>0.02032</length>
           </cylinder>
         </geometry>
       </collision>
-      <xacro:cylinder_inertia m="0.125" r="0.0508" h="0.055"/>
+      <xacro:cylinder_inertia m="0.125" r="0.021" h="0.02032"/>
       <sensor name="lidar" type="gpu_lidar">
         <always_on>true</always_on>
@@ -321,5 +232,5 @@
       <parent>base_link</parent>
       <child>camera_link</child>
-      <pose relative_to="base_link">0.215 0 0.05 0 0 0</pose>
+      <pose relative_to="base_link">0.05715 0 0.01 0 0 0</pose>
     </joint>
     <link name='camera_link'>
@@ -328,5 +239,5 @@
         <geometry>
           <box><size>
-            0.015 0.130 0.0222
+            0.015 0.030 0.0222
           </size></box>
         </geometry>
@@ -335,9 +246,9 @@
         <geometry>
           <box><size>
-            0.015 0.130 0.0222
-          </size></box>
-        </geometry>
-      </collision>
-      <xacro:box_inertia m="0.035" w="0.015" d="0.130" h="0.0222"/>
+            0.015 0.030 0.0222
+          </size></box>
+        </geometry>
+      </collision>
+      <xacro:box_inertia m="0.035" w="0.015" d="0.030" h="0.0222"/>
       <sensor name="depth_camera" type="rgbd_camera">
         <always_on>true</always_on>

Commit message: Add simulation launch file for HERMES navigation and exploration stack

File: urdf/hermes_sim.sdf.xacro (robot description, xacro)
@@ -229,58 +229,4 @@
       </sensor>
     </link>
-    <joint name="camera_joint" type="fixed">
-      <parent>base_link</parent>
-      <child>camera_link</child>
-      <pose relative_to="base_link">0.05715 0 0.01 0 0 0</pose>
-    </joint>
-    <link name='camera_link'>
-      <pose relative_to="camera_joint"/>
-      <visual name="camera_link_visual">
-        <geometry>
-          <box><size>
-            0.015 0.030 0.0222
-          </size></box>
-        </geometry>
-      </visual>
-      <collision name="camera_link_collision">
-        <geometry>
-          <box><size>
-            0.015 0.030 0.0222
-          </size></box>
-        </geometry>
-      </collision>
-      <xacro:box_inertia m="0.035" w="0.015" d="0.030" h="0.0222"/>
-      <sensor name="depth_camera" type="rgbd_camera">
-        <always_on>true</always_on>
-        <visualize>true</visualize>
-        <update_rate>5.0</update_rate>
-        <topic>depth_camera</topic>
-        <gz:frame_id>camera_link</gz:frame_id>
-        <camera>
-          <horizontal_fov>1.047198</horizontal_fov>
-          <image>
-            <width>640</width>
-            <height>480</height>
-          </image>
-          <clip>
-            <near>0.05</near>
-            <far>3</far>
-          </clip>
-        </camera>
-        <baseline>0.2</baseline>
-        <pointCloudCutoff>0.5</pointCloudCutoff>
-        <pointCloudCutoffMax>3.0</pointCloudCutoffMax>
-        <distortionK1>0</distortionK1>
-        <distortionK2>0</distortionK2>
-        <distortionK3>0</distortionK3>
-        <distortionT1>0</distortionT1>
-        <distortionT2>0</distortionT2>
-        <CxPrime>0</CxPrime>
-        <Cx>0</Cx>
-        <Cy>0</Cy>
-        <focalLength>0</focalLength>
-        <hackBaseline>0</hackBaseline>
-      </sensor>
-    </link>
   </model>
 </sdf>

Commit message: refactor: add EKF configuration and integrate with navigation stack; update simulation parameters for improved performance

File: urdf/hermes_sim.sdf.xacro (robot description, xacro)
@@ -4,5 +4,5 @@
     <!-- Define robot constants -->
     <xacro:property name="base_width" value="0.1143"/>
-    <xacro:property name="base_length" value="0.1143"/>
+    <xacro:property name="base_length" value="0.14"/>
     <xacro:property name="base_height" value="0.0762"/>
     <xacro:property name="wheel_radius" value="0.03302"/>
@@ -10,5 +10,5 @@
     <xacro:property name="wheel_ygap" value="0.01"/>
     <xacro:property name="wheel_zoff" value="0.01778"/>
-    <xacro:property name="wheel_xoff" value="0.03"/>
+    <xacro:property name="wheel_xoff" value="0.035"/>
     <xacro:property name="caster_xoff" value="0.04"/>
     <!-- Define some commonly used intertial properties  -->
@@ -177,4 +177,11 @@
       <!-- input -->
       <topic>/demo/cmd_vel</topic>
+      <!-- odometry output -->
+      <odom_topic>/model/hermes/odometry</odom_topic>
+      <odom_publish_frequency>30</odom_publish_frequency>
+      <frame_id>odom</frame_id>
+      <child_frame_id>base_link</child_frame_id>
+      <!-- Disable TF publishing — robot_localization EKF publishes odom→base_link -->
+      <tf_topic></tf_topic>
     </plugin>
     <plugin
